Commit message: able to get transform from aruco tag to base link. Still need to fix rotation tho

File: jellyfish_gazebo/dji_m210_description/urdf/gimbal/gimbal.xacro (robot description, xacro)
@@ -97,33 +97,4 @@
             </visual>
         </link>
-        <!-- Mount a generic odometry sensor providing ground truth. -->
-        <xacro:odometry_plugin_macro
-            namespace="${namespace}/gimbal_ground_truth"
-            odometry_sensor_suffix=""
-            parent_link="gimbal_yaw_link"
-            pose_topic="pose"
-            pose_with_covariance_topic="pose_with_covariance"
-            position_topic="position"
-            transform_topic="transform"
-            odometry_topic="odometry"
-            parent_frame_id="world"
-            mass_odometry_sensor="0.00001"
-            measurement_divisor="1"
-            measurement_delay="0"
-            unknown_delay="0.0"
-            noise_normal_position="0 0 0"
-            noise_normal_quaternion="0 0 0"
-            noise_normal_linear_velocity="0 0 0"
-            noise_normal_angular_velocity="0 0 0"
-            noise_uniform_position="0 0 0"
-            noise_uniform_quaternion="0 0 0"
-            noise_uniform_linear_velocity="0 0 0"
-            noise_uniform_angular_velocity="0 0 0"
-            enable_odometry_map="false"
-            odometry_map=""
-            image_scale="">
-            <inertia ixx="0.00001" ixy="0.0" ixz="0.0" iyy="0.00001" iyz="0.0" izz="0.00001" /> <!-- [kg.m^2] [kg.m^2] [kg.m^2] [kg.m^2] [kg.m^2] [kg.m^2] -->
-            <origin xyz="0.0 0.0 0.0" rpy="0.0 0.0 0.0" />
-        </xacro:odometry_plugin_macro>
         <gazebo>
             <plugin name="gazebo_ros_control" filename="libgazebo_ros_control.so">
