Commit message: Fix python3 incompatibility and namespaces

File: jellyfish_gazebo/jellyfish_sim/URDF/basic_tag.xacro (robot description, xacro)
@@ -13,5 +13,5 @@
         <visual>
             <geometry>
-                <mesh filename="package://dji_m210_gazebo/meshes/tag14/tag14.dae"/>
+                <mesh filename="package://jellyfish_sim/meshes/tag14/tag14.dae"/>
             </geometry>
         </visual>

Commit message: Add vrx buoyancy plugin for landing platform

File: jellyfish_gazebo/jellyfish_sim/URDF/basic_tag.xacro (robot description, xacro)
@@ -18,5 +18,5 @@
         <collision>
             <geometry>
-                <box size="1 1 0.05"/>
+                <box size="2 2 0.05"/>
             </geometry>
         </collision>
@@ -54,3 +54,21 @@
         <origin xyz="0.0 0.0 0.0" rpy="0.0 0.0 0.0" />
     </xacro:odometry_plugin_macro>
+    <gazebo>
+        <plugin name="LandingPlatformBuoyancyPlugin" filename="libbuoyancy_gazebo_plugin.so">
+        <wave_model>ocean_waves</wave_model>
+        <fluid_density>1000</fluid_density>
+        <fluid_level>0.0</fluid_level>
+        <linear_drag>1000</linear_drag>
+        <angular_drag>200</angular_drag>
+        <buoyancy name="buoyancy_base">
+            <link_name>base_link</link_name>
+            <pose>0 0 -0.1 0 0 0</pose>
+            <geometry>
+                <box>
+                    <size>1 1 0.05</size>
+                </box>
+            </geometry>
+        </buoyancy>
+        </plugin>
+    </gazebo>
 </robot>
