Commit message: added gimbal and marvelmind works in HITL sim. Modified simulate launch files

File: jellyfish_gazebo/dji_m210_description/urdf/HITL_dji_m210.xacro (robot description, xacro)
@@ -3,18 +3,24 @@
 	<xacro:include filename="$(find dji_m210_description)/urdf/component_snippets.xacro"/>
 	<xacro:include filename="$(find dji_m210_description)/urdf/gimbal/gimbal.xacro"/>
-  <!-- Arguments -->
-  <xacro:arg name="hitl_model" default="true"/>
-  <!-- Properties -->
-  <xacro:property name="mass" value="2.355" /> <!-- [kg] -->
-  <xacro:property name="mass_rotor" value="0.08" /> <!-- [kg] -->
-  <xacro:property name="arm_length" value="0.17" /> <!-- [m] -->
-  <xacro:property name="rotor_offset_top" value="0.1" /> <!-- [m] -->
-  <xacro:property name="radius_rotor" value="0.195" /> <!-- [m] -->
-  <xacro:property name="sin30" value="0.5" />
-  <xacro:property name="cos30" value="0.866025403784" />
-  <xacro:property name="sqrt2" value="1.4142135623730951" />
+	<!-- Arguments -->
+	<xacro:arg name="hitl_model" default="true"/>
+	<!-- Properties -->
+	<xacro:property name="mass" value="2.355" /> <!-- [kg] -->
+	<xacro:property name="mass_rotor" value="0.08" /> <!-- [kg] -->
+	<xacro:property name="arm_length" value="0.17" /> <!-- [m] -->
+	<xacro:property name="rotor_offset_top" value="0.1" /> <!-- [m] -->
+	<xacro:property name="radius_rotor" value="0.195" /> <!-- [m] -->
+	<xacro:property name="sin30" value="0.5" />
+	<xacro:property name="cos30" value="0.866025403784" />
+	<xacro:property name="sqrt2" value="1.4142135623730951" />
 	<xacro:property name="body_width" value="0.3" />
-  <xacro:property name="body_height" value="0.16" />
-  <!-- Property Blocks -->
+	<xacro:property name="body_height" value="0.16" />
+	<xacro:property name="gimbal_roll_min_angle" value="-0.45" />
+	<xacro:property name="gimbal_roll_max_angle" value="0.45" />
+	<xacro:property name="gimbal_pitch_min_angle" value="-1.57" />
+	<xacro:property name="gimbal_pitch_max_angle" value="1.57" />
+	<xacro:property name="gimbal_yaw_min_angle" value="-1.57" />
+	<xacro:property name="gimbal_yaw_max_angle" value="1.57" />
+  	<!-- Property Blocks -->
 	<!-- materials -->
 	<material name="black">
@@ -171,4 +177,11 @@
 	</gazebo>
 	<!--Slap on a gimbal and a camera-->
-	<xacro:dji_m210_gimbal/>
+	<xacro:dji_m210_gimbal
+		gimbal_roll_min_angle="${gimbal_roll_min_angle}"
+		gimbal_roll_max_angle="${gimbal_roll_max_angle}"
+		gimbal_pitch_min_angle="${gimbal_pitch_min_angle}"
+		gimbal_pitch_max_angle="${gimbal_pitch_max_angle}"
+		gimbal_yaw_min_angle="${gimbal_yaw_min_angle}"
+		gimbal_yaw_max_angle="${gimbal_yaw_max_angle}"
+		/>
 </robot>

File: jellyfish_gazebo/dji_m210_description/urdf/SITL_dji_m210.xacro (robot description, xacro)
@@ -43,4 +43,10 @@
   <xacro:property name="color" value="DarkGrey" />
   <xacro:property name="sqrt2" value="1.4142135623730951" />
+  <xacro:property name="gimbal_roll_min_angle" value="-0.45" />
+  <xacro:property name="gimbal_roll_max_angle" value="0.45" />
+  <xacro:property name="gimbal_pitch_min_angle" value="-1.57" />
+  <xacro:property name="gimbal_pitch_max_angle" value="1.57" />
+  <xacro:property name="gimbal_yaw_min_angle" value="-1.57" />
+  <xacro:property name="gimbal_yaw_max_angle" value="1.57" />
   <!-- Property Blocks -->
   <xacro:property name="body_inertia">
@@ -218,4 +224,11 @@
   </gazebo>
 	<!--Slap on a gimbal and a camera-->
-	<xacro:dji_m210_gimbal/>
+	<xacro:dji_m210_gimbal
+		gimbal_roll_min_angle="${gimbal_roll_min_angle}"
+		gimbal_roll_max_angle="${gimbal_roll_max_angle}"
+		gimbal_pitch_min_angle="${gimbal_pitch_min_angle}"
+		gimbal_pitch_max_angle="${gimbal_pitch_max_angle}"
+		gimbal_yaw_min_angle="${gimbal_yaw_min_angle}"
+		gimbal_yaw_max_angle="${gimbal_yaw_max_angle}"
+		/>
 </robot>

File: jellyfish_gazebo/dji_m210_description/urdf/gimbal/gimbal.xacro (robot description, xacro)
@@ -3,5 +3,5 @@
     <xacro:include filename="$(find dji_m210_description)/urdf/gimbal/gimbal_joints.xacro"/>
     <xacro:property name="M_PI" value="3.14"/>
-    <xacro:macro name="dji_m210_gimbal">
+    <xacro:macro name="dji_m210_gimbal" params="gimbal_roll_min_angle gimbal_roll_max_angle gimbal_pitch_min_angle gimbal_pitch_max_angle gimbal_yaw_min_angle gimbal_yaw_max_angle">
         <joint name="gimbal_base_joint" type="fixed">
             <parent link="base_link"/>
@@ -37,6 +37,6 @@
             parent="gimbal_base_plate"
             child="gimbal_roll_link"
-            lower_limit="-0.48"
-            upper_limit="0.48"
+            lower_limit="${gimbal_roll_min_angle}"
+            upper_limit="${gimbal_roll_max_angle}"
             axis_xyz="1 0 0"
             origin_xyz="0.05 0 -0.04"
@@ -58,6 +58,6 @@
             parent="gimbal_roll_link"
             child="gimbal_pitch_link"
-            lower_limit="-0.48"
-            upper_limit="0.48"
+            lower_limit="${gimbal_pitch_min_angle}"
+            upper_limit="${gimbal_pitch_max_angle}"
             axis_xyz="0 1 0"
             origin_xyz="0 0 0"
@@ -79,6 +79,6 @@
             parent="gimbal_pitch_link"
             child="gimbal_yaw_link"
-            lower_limit="-1.57"
-            upper_limit="1.57"
+            lower_limit="${gimbal_yaw_min_angle}"
+            upper_limit="${gimbal_yaw_max_angle}"
             axis_xyz="0 0 1"
             origin_xyz="0 0 0"
@@ -97,4 +97,33 @@
             </visual>
         </link>
+        <!-- Mount a generic odometry sensor providing ground truth. -->
+        <xacro:odometry_plugin_macro
+            namespace="${namespace}/gimbal_ground_truth"
+            odometry_sensor_suffix=""
+            parent_link="gimbal_yaw_link"
+            pose_topic="pose"
+            pose_with_covariance_topic="pose_with_covariance"
+            position_topic="position"
+            transform_topic="transform"
+            odometry_topic="odometry"
+            parent_frame_id="world"
+            mass_odometry_sensor="0.00001"
+            measurement_divisor="1"
+            measurement_delay="0"
+            unknown_delay="0.0"
+            noise_normal_position="0 0 0"
+            noise_normal_quaternion="0 0 0"
+            noise_normal_linear_velocity="0 0 0"
+            noise_normal_angular_velocity="0 0 0"
+            noise_uniform_position="0 0 0"
+            noise_uniform_quaternion="0 0 0"
+            noise_uniform_linear_velocity="0 0 0"
+            noise_uniform_angular_velocity="0 0 0"
+            enable_odometry_map="false"
+            odometry_map=""
+            image_scale="">
+            <inertia ixx="0.00001" ixy="0.0" ixz="0.0" iyy="0.00001" iyz="0.0" izz="0.00001" /> <!-- [kg.m^2] [kg.m^2] [kg.m^2] [kg.m^2] [kg.m^2] [kg.m^2] -->
+            <origin xyz="0.0 0.0 0.0" rpy="0.0 0.0 0.0" />
+        </xacro:odometry_plugin_macro>
         <gazebo>
             <plugin name="gazebo_ros_control" filename="libgazebo_ros_control.so">

Commit message: update jellyfish_sim based on code in bbuav_gazebo_plugins allow the drone to float on water increate the collision size of the drone body for more stability improve the use of namespace for landing platform and drone implement dji_sdk stop and start service call replace use of mav_msgs CommandTrajectory by the Catersian action goal

File: jellyfish_gazebo/dji_m210_description/urdf/HITL_dji_m210.xacro (robot description, xacro)
@@ -178,4 +178,5 @@
 	<!--Slap on a gimbal and a camera-->
 	<xacro:dji_m210_gimbal
+		namespace="${namespace}"
 		gimbal_roll_min_angle="${gimbal_roll_min_angle}"
 		gimbal_roll_max_angle="${gimbal_roll_max_angle}"

File: jellyfish_gazebo/dji_m210_description/urdf/SITL_dji_m210.xacro (robot description, xacro)
@@ -20,7 +20,10 @@
   <xacro:include filename="$(find dji_m210_description)/urdf/component_snippets.xacro"/>
   <xacro:include filename="$(find dji_m210_description)/urdf/gimbal/gimbal.xacro"/>
+  <xacro:arg name="namespace" default="dji_m210" />
+  <xacro:arg name="dji_sdk_ns" default="dji_sdk" />
   <!-- Properties -->
-  <xacro:property name="namespace" value="dji_m210" />
-  <xacro:property name="rotor_velocity_slowdown_sim" value="10" />
+  <xacro:property name="namespace" value="$(arg namespace)" />
+  <xacro:property name="dji_sdk_ns" value="$(arg dji_sdk_ns)" />
+  <xacro:property name="rotor_velocity_slowdown_sim" value="5" />
   <xacro:property name="mesh_file" value="package://dji_m210_description/meshes/dji_m210/dji_m210_flipped_rotorless.dae" />
   <xacro:property name="mesh_scale" value="1 1 1"/>
@@ -28,6 +31,6 @@
   <xacro:property name="mesh_scale_prop" value=".12 .12 .12"/>
   <xacro:property name="mass" value="2.355" /> <!-- [kg] -->
-  <xacro:property name="body_width" value="0.3" /> <!-- [m] -->
-  <xacro:property name="body_height" value="0.16" /> <!-- [m] -->
+  <xacro:property name="body_width" value="0.50" /> <!-- [m] -->
+  <xacro:property name="body_height" value="0.2" /> <!-- [m] -->
   <xacro:property name="mass_rotor" value="0.08" /> <!-- [kg] -->
   <xacro:property name="arm_length" value="0.17" /> <!-- [m] -->
@@ -201,5 +204,5 @@
       <topic>__default_topic__</topic>
       <plugin filename="libgazebo_ros_imu_sensor.so" name="imu_plugin">
-        <topicName>/dji_sdk/imu</topicName>
+        <topicName>${dji_sdk_ns}/imu</topicName>
         <bodyName>imu_link</bodyName>
         <updateRateHZ>10.0</updateRateHZ>
@@ -219,10 +222,11 @@
       <commandRateThrustSubTopic>command/rate</commandRateThrustSubTopic>
       <commandMotorSpeedSubTopic>command/motor_speed</commandMotorSpeedSubTopic>
-      <imuSubTopic>dji_sdk/imu</imuSubTopic>
-      <motorSpeedCommandPubTopic>gazebo/command/motor_speed</motorSpeedCommandPubTopic>
+      <imuSubTopic>${dji_sdk_ns}/imu</imuSubTopic>
+      <motorSpeedCommandPubTopic>gazebo_command/motor_speed</motorSpeedCommandPubTopic>
     </plugin>
   </gazebo>
 	<!--Slap on a gimbal and a camera-->
 	<xacro:dji_m210_gimbal
+    namespace="${namespace}"
 		gimbal_roll_min_angle="${gimbal_roll_min_angle}"
 		gimbal_roll_max_angle="${gimbal_roll_max_angle}"

File: jellyfish_gazebo/dji_m210_description/urdf/gimbal/gimbal.xacro (robot description, xacro)
@@ -3,5 +3,6 @@
     <xacro:include filename="$(find dji_m210_description)/urdf/gimbal/gimbal_joints.xacro"/>
     <xacro:property name="M_PI" value="3.14"/>
-    <xacro:macro name="dji_m210_gimbal" params="gimbal_roll_min_angle gimbal_roll_max_angle gimbal_pitch_min_angle gimbal_pitch_max_angle gimbal_yaw_min_angle gimbal_yaw_max_angle">
+    <xacro:macro name="dji_m210_gimbal" params="namespace gimbal_roll_min_angle gimbal_roll_max_angle gimbal_pitch_min_angle gimbal_pitch_max_angle gimbal_yaw_min_angle gimbal_yaw_max_angle">
+        <xacro:arg name="namespace" default="dji_m210" />
         <joint name="gimbal_base_joint" type="fixed">
             <parent link="base_link"/>
@@ -108,5 +109,5 @@
                 <update_rate>10</update_rate>
                 <camera>
-					<pose>0.107 0 -0.227 0 0 0</pose>
+					<pose>0.107 0 0 0 0 0</pose>
 					<horizontal_fov>${94 * M_PI/180.0}</horizontal_fov>
 					<image>
@@ -124,6 +125,6 @@
                 <alwaysOn>true</alwaysOn>
                 <updateRate>10</updateRate>
-                <imageTopicName>dji_sdk/image_raw</imageTopicName>
-                <cameraInfoTopicName>dji_sdk/camera_info</cameraInfoTopicName>
+                <imageTopicName>${namespace}/image_raw</imageTopicName>
+                <cameraInfoTopicName>${namespace}/camera_info</cameraInfoTopicName>
                 <frameName>gimbal_yaw_link</frameName>
                 </plugin>

File: jellyfish_gazebo/dji_m210_description/urdf/multirotor_base.xacro (robot description, xacro)
@@ -27,5 +27,5 @@
         <origin xyz="0 0 0" rpy="0 0 0" />
         <geometry>
-            <box size="${body_width} ${body_width} ${body_height}" /> <!-- [m] [m] [m] -->
+            <box size="${body_width} ${body_width} ${body_height}" /> [m] [m] [m]
         </geometry>
         </collision>
@@ -37,4 +37,23 @@
         <linkName>base_link</linkName>
         <rotorVelocitySlowdownSim>${rotor_velocity_slowdown_sim}</rotorVelocitySlowdownSim>
+        </plugin>
+    </gazebo>
+    <gazebo>
+        <plugin name="BuoyancyPlugin" filename="libbuoyancy_gazebo_plugin.so">
+        <fluid_density>200</fluid_density>
+        <linear_drag>100</linear_drag>
+        <angular_drag>20</angular_drag>
+        <buoyancy name="buoyancy_base">
+            <link_name>base_link</link_name>
+            <pose>0 0 -0.1 0 0 0</pose>
+            <geometry>
+                <box>
+                    <size>0.4 0.4 0.2</size>
+                </box>
+            </geometry>
+        </buoyancy>
+        <link name="body">
+        <volume>100</volume>
+        </link>
         </plugin>
     </gazebo>

File: jellyfish_gazebo/jellyfish_sim/URDF/basic_tag.xacro (robot description, xacro)
@@ -1,7 +1,10 @@
 <?xml version="1.0"?>
 <robot name="aruco_tag" xmlns:xacro="http://ros.org/wiki/xacro">
+    <xacro:include filename="$(find wave_gazebo)/world_models/ocean_waves/model.xacro"/>
     <xacro:include filename="$(find dji_m210_description)/urdf/component_snippets.xacro"/>
+    <xacro:arg name="use_buoyancy" default="false" />
+    <xacro:arg name="namespace" default="landing_platform" />
     <!-- Properties -->
-    <xacro:property name="namespace" value="landing_platform" />
+    <xacro:property name="namespace" value="$(arg namespace)" />
     <link name="base_link"></link>
     <joint name="base_joint" type="fixed">
@@ -18,5 +21,5 @@
         <collision>
             <geometry>
-                <box size="2 2 0.05"/>
+                <box size="1 1 0.1"/>
             </geometry>
         </collision>
@@ -54,21 +57,23 @@
         <origin xyz="0.0 0.0 0.0" rpy="0.0 0.0 0.0" />
     </xacro:odometry_plugin_macro>
-    <gazebo>
-        <plugin name="LandingPlatformBuoyancyPlugin" filename="libbuoyancy_gazebo_plugin.so">
-        <wave_model>ocean_waves</wave_model>
-        <fluid_density>1000</fluid_density>
-        <fluid_level>0.0</fluid_level>
-        <linear_drag>1000</linear_drag>
-        <angular_drag>200</angular_drag>
-        <buoyancy name="buoyancy_base">
-            <link_name>base_link</link_name>
-            <pose>0 0 -0.1 0 0 0</pose>
-            <geometry>
-                <box>
-                    <size>1 1 0.05</size>
-                </box>
-            </geometry>
-        </buoyancy>
-        </plugin>
-    </gazebo>
+    <xacro:if value="$(arg use_buoyancy)">
+        <gazebo>
+            <plugin name="LandingPlatformBuoyancyPlugin" filename="libbuoyancy_gazebo_plugin.so">
+            <wave_model>ocean_waves</wave_model>
+            <fluid_density>5000</fluid_density>
+            <fluid_level>0.0</fluid_level>
+            <linear_drag>1000</linear_drag>
+            <angular_drag>200</angular_drag>
+            <buoyancy name="buoyancy_base">
+                <link_name>base_link</link_name>
+                <pose>0 0 -0.2 0 0 0</pose>
+                <geometry>
+                    <box>
+                        <size>2 2 0.3</size>
+                    </box>
+                </geometry>
+            </buoyancy>
+            </plugin>
+        </gazebo>
+    </xacro:if>
 </robot>
