Commit message: fix some parameters so the uav doesn't break as often default enable motors

File: jellyfish_gazebo/dji_m210_description/urdf/multirotor_base.xacro (robot description, xacro)
@@ -19,6 +19,5 @@
         <origin xyz="0 0 0" rpy="0 0 0" />
         <geometry>
-            <mesh filename="${mesh_file}"
-            scale="${mesh_scale}" />
+            <mesh filename="${mesh_file}" scale="${mesh_scale}" />
             <!-- <box size="${body_width} ${body_width} ${body_height}"/> --> <!-- [m] [m] [m] -->
         </geometry>
@@ -27,5 +26,6 @@
         <origin xyz="0 0 0" rpy="0 0 0" />
         <geometry>
-            <box size="${body_width} ${body_width} ${body_height}" /> [m] [m] [m]
+            <!-- [m] [m] [m] -->
+            <box size="${body_width} ${body_width} ${body_height}" />
         </geometry>
         </collision>
@@ -41,10 +41,10 @@
     <gazebo>
         <plugin name="BuoyancyPlugin" filename="libbuoyancy_gazebo_plugin.so">
-        <fluid_density>200</fluid_density>
+        <fluid_density>997</fluid_density>
         <linear_drag>100</linear_drag>
         <angular_drag>20</angular_drag>
         <buoyancy name="buoyancy_base">
             <link_name>base_link</link_name>
-            <pose>0 0 -0.1 0 0 0</pose>
+            <pose>0 0 -0.03 0 0 0</pose>
             <geometry>
                 <box>

File: jellyfish_gazebo/jellyfish_urdf/URDF/basic_tag.xacro (robot description, xacro)
@@ -61,5 +61,5 @@
             <plugin name="LandingPlatformBuoyancyPlugin" filename="libbuoyancy_gazebo_plugin.so">
             <wave_model>ocean_waves</wave_model>
-            <fluid_density>5000</fluid_density>
+            <fluid_density>997</fluid_density>
             <fluid_level>0.0</fluid_level>
             <linear_drag>1000</linear_drag>
@@ -67,8 +67,8 @@
             <buoyancy name="buoyancy_base">
                 <link_name>base_link</link_name>
-                <pose>0 0 -0.2 0 0 0</pose>
+                <pose>0 0 -0.4 0 0 0</pose>
                 <geometry>
                     <box>
-                        <size>2 2 0.3</size>
+                        <size>1 1 0.3</size>
                     </box>
                 </geometry>
