Commit message: rename jellyfish_sim to jellyfish_urdf

File: jellyfish_gazebo/jellyfish_urdf/URDF/basic_tag.xacro (robot description, xacro)
@@ -16,5 +16,5 @@
         <visual>
             <geometry>
-                <mesh filename="package://jellyfish_sim/meshes/tag14/tag14.dae"/>
+                <mesh filename="package://jellyfish_urdf/meshes/tag14/tag14.dae"/>
             </geometry>
         </visual>
